File: Hardware/power.sch (KiCad schematic (older format))
At the start: 25 parts, among them IC201 FT232RQ, P201 USB_OTG, P202 POWER, P203 3V3, U201 MCP1700T-3302E/TT

Commit message: more layout
Parts:
- removed P203: 3V3, Pin_Headers:Pin_Header_Straight_1x02, symbol CONN_01X02
Changed lines of the file:
@@
 Connection ~ 4950 3525
 Connection ~ 4810 3525
-$Comp
-L CONN_01X02 P203
-U 1 1 591371DE
-P 8225 1040
-F 0 "P203" H 8225 1190 50  0000 C CNN
-F 1 "3V3" V 8325 1040 50  0000 C CNN
-F 2 "Pin_Headers:Pin_Header_Straight_1x02" H 8225 1040 50  0001 C CNN
-F 3 "" H 8225 1040 50  0000 C CNN
-F 4 "Value" H 8225 1040 60  0001 C CNN "Fieldname"
-	1    8225 1040
-	0    -1   -1   0
-$EndComp
-Wire Wire Line
-	8175 1240 8175 1480
-Connection ~ 8175 1480
-$Comp
-L GND #PWR021
-U 1 1 59137A62
-P 8275 1285
-F 0 "#PWR021" H 8275 1035 50  0001 C CNN
-F 1 "GND" H 8275 1135 50  0000 C CNN
-F 2 "" H 8275 1285 50  0000 C CNN
-F 3 "" H 8275 1285 50  0000 C CNN
-	1    8275 1285
-	1    0    0    -1
-$EndComp
-Wire Wire Line
-	8275 1240 8275 1285
 $EndSCHEMATC

Commit message: moved headers from power side of boards and rerouted traces
Parts:
- IC201: footprint Housings_DFN_QFN:QFN-32-1EP_5x5mm_Pitch0.5mm -> CentralCommand:FT232RQ
Changed lines of the file:
@@
 F 0 "IC201" H 5790 5865 50  0000 C CNN
 F 1 "FT232RQ" H 6790 3905 50  0000 C CNN
-F 2 "Housings_DFN_QFN:QFN-32-1EP_5x5mm_Pitch0.5mm" H 6340 4615 50  0001 C CIN
+F 2 "CentralCommand:FT232RQ" H 6340 4615 50  0001 C CIN
 F 3 "http://www.ftdichip.com/Support/Documents/DataSheets/ICs/DS_FT232R.pdf" H 6340 4615 50  0001 C CNN
 F 4 "Value" H 6340 4615 60  0001 C CNN "Fieldname"
